File: macos/docs/pcb/blinker.kicad_pcb (KiCad board)
At the start: 2 copper layers, 38 x 38 mm, 11 parts, among them J1 Power 9 V, Q1 2N3904 (or any small NPN), Q2 2N3904 (or any small NPN)

Commit message: An open board found by its folder as well as its name; a wire's net highlighted in KiCad; boards kept through renames
- KiCad's open board is the circuit's only when its project's folder is the board file's (links followed, as /tmp is
  /private/tmp on a Mac). Matching on the file name alone, an update went to another project's board of the same name
  open in KiCad. Test.
- Selecting wires of one net in the schematic highlights the net in KiCad's PCB editor ($NET on port 4242, as KiCad's
  schematic editor does): the board's name for each wire's net (PCBNetlistBuilder's wireNets, from the extractor's
  nets). Checked in KiCad 10.0.7's editor. Test.
- A transistor's value on the board is its part number ("2N3904"), not the breadboard's buying note.
- A circuit renamed or saved as another file keeps its board (PCBDesign.board), in the app and in jspice-mcp.
- The docs' board brought up to date with that (two values), still clean in KiCad's DRC.

Co-Authored-By: Claude Opus 5.5 <noreply@anthropic.com>
Claude-Session: https://claude.ai/code/session_013QXdZmcGP1CYZDQFYYtfKg
Parts:
- Q1, Q2: value 2N3904 (or any small NPN) -> 2N3904
Changed lines of the file:
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@@
 			)
 		)
-		(property "Value" "2N3904 (or any small NPN)"
+		(property "Value" "2N3904"
 			(at 1.27 2.79 0)
 			(layer "F.Fab")
@@
 			)
 		)
-		(property "Value" "2N3904 (or any small NPN)"
+		(property "Value" "2N3904"
 			(at 1.27 2.79 0)
 			(layer "F.Fab")
